File: PR-4PP.kicad_pcb (KiCad board)
At the start: 2 copper layers, 84.1 x 38.1 mm, 36 parts, among them SW1 SW_Push, U1 ATmega32U4-AU, U3 SRV05-4, Y1 16mHz

Commit message: small changes
Parts:
- turned F1 to 90 degrees
Connections:
- F1 pad 1: VBUS -> +5V
- F1 pad 2: +5V -> VBUS
Routing:
- removed copper zone on B.Cu, net (none)
