File: PR-4PP.sch (KiCad schematic (older format))
At the start: 28 parts, among them SW1 SW_Push, U1 ATmega32U4-AU, U3 SRV05-4, Y1 16mHz

Commit message: reroute usb
Parts:
- USB1: footprint (none) -> Type-C:HRO-TYPE-C-31-M-12-HandSoldering
Connections:
- no-connect marks 26 -> 24
Changed lines of the file:
@@
 Text GLabel 1750 1800 2    50   Input ~ 0
 D+
-Text GLabel 3700 1950 0    50   Input ~ 0
+Text GLabel 5100 2150 2    50   Input ~ 0
+D-
+Text GLabel 3650 1950 0    50   Input ~ 0
 D+
 Wire Wire Line
-	3700 1950 3900 1950
-Text GLabel 5150 2150 2    50   Input ~ 0
-D-
-Wire Wire Line
-	5150 2150 4900 2150
-NoConn ~ 4900 1950
-NoConn ~ 3900 2150
+	3650 1950 3900 1950
 $Comp
 L power:GNDPWR #PWR0118
@@
 F 0 "USB1" H 1200 2300 60  0000 C CNN
 F 1 "HRO-TYPE-C-31-M-12" V 1000 1600 60  0000 C CNN
-F 2 "" H 1400 1650 60  0001 C CNN
+F 2 "Type-C:HRO-TYPE-C-31-M-12-HandSoldering" H 1400 1650 60  0001 C CNN
 F 3 "" H 1400 1650 60  0001 C CNN
 	1    1400 1650
@@
 	0    1    1    0
 $EndComp
+Wire Wire Line
+	5100 2150 4900 2150
 $EndSCHEMATC

Commit message: reroute & fillzones
Parts:
- MX1, MX2, MX3: footprint MX_Alps_Hybrid:MX-1U-NoLED -> MX_Only:MXOnly-1U-Hotswap-Antishear
- MX4: footprint MX_Alps_Hybrid:MX-1U -> MX_Only:MXOnly-1U-Hotswap-Antishear
Connections:
- net DR-: now reaches R3.1, U1.3 (D-)
- net DR+: now reaches R2.1, U1.4 (D+)
Changed lines of the file:
@@
 F 0 "MX1" H 9583 3423 60  0000 C CNN
 F 1 "MX-NoLED" H 9583 3349 20  0000 C CNN
-F 2 "MX_Alps_Hybrid:MX-1U-NoLED" H 8925 3175 60  0001 C CNN
+F 2 "MX_Only:MXOnly-1U-Hotswap-Antishear" H 8925 3175 60  0001 C CNN
 F 3 "" H 8925 3175 60  0001 C CNN
 	1    9550 3200
@@
 F 0 "MX3" H 9583 4173 60  0000 C CNN
 F 1 "MX-NoLED" H 9583 4099 20  0000 C CNN
-F 2 "MX_Alps_Hybrid:MX-1U-NoLED" H 8925 3925 60  0001 C CNN
+F 2 "MX_Only:MXOnly-1U-Hotswap-Antishear" H 8925 3925 60  0001 C CNN
 F 3 "" H 8925 3925 60  0001 C CNN
 	1    9550 3950
@@
 F 0 "MX2" H 10483 3423 60  0000 C CNN
 F 1 "MX-NoLED" H 10483 3349 20  0000 C CNN
-F 2 "MX_Alps_Hybrid:MX-1U-NoLED" H 9825 3175 60  0001 C CNN
+F 2 "MX_Only:MXOnly-1U-Hotswap-Antishear" H 9825 3175 60  0001 C CNN
 F 3 "" H 9825 3175 60  0001 C CNN
 	1    10450 3200
@@
 F 0 "MX4" H 10483 4173 60  0000 C CNN
 F 1 "MX-NoLED" H 10483 4099 20  0000 C CNN
-F 2 "MX_Alps_Hybrid:MX-1U" H 9825 3925 60  0001 C CNN
+F 2 "MX_Only:MXOnly-1U-Hotswap-Antishear" H 9825 3925 60  0001 C CNN
 F 3 "" H 9825 3925 60  0001 C CNN
 	1    10450 3950
@@
 Wire Wire Line
 	5100 2150 4900 2150
+Text Label 6900 3750 0    50   ~ 0
+DR+
+Text Label 6900 3850 0    50   ~ 0
+DR-
 $EndSCHEMATC

Commit message: add silkscreen and part numbers
Parts:
- added H1, H2, H3, H4, H5, H6: MountingHole, MountingHole:MountingHole_2mm, symbol Mechanical:MountingHole
- C1, C2: LCSC (none) -> C1804
- C3: LCSC (none) -> C28323
- C4, C5, C6: LCSC (none) -> C49678
- C7: LCSC (none) -> C15850
- D1, D2, D3, D4: LCSC (none) -> C64898
- F1: LCSC (none) -> C70076
- L1: LCSC (none) -> C1017
- R1: LCSC (none) -> C25804
- R2, R3: LCSC (none) -> C17561
- R4: LCSC (none) -> C17414
- R5, R6: LCSC (none) -> C23186
- SW1: LCSC (none) -> C318884
- U1: LCSC (none) -> C44854
- U3: LCSC (none) -> C85364
- USB1: LCSC (none) -> C165948
- Y1: LCSC (none) -> C13738
Connections:
- no-connect marks 24 -> 26
Changed lines of the file:
@@
 F 2 "Package_QFP:TQFP-44_10x10mm_P0.8mm" H 7650 4250 50  0001 C CIN
 F 3 "http://ww1.microchip.com/downloads/en/DeviceDoc/Atmel-7766-8-bit-AVR-ATmega16U4-32U4_Datasheet.pdf" H 7650 4250 50  0001 C CNN
+F 4 "C44854" H 7650 4250 50  0001 C CNN "LCSC"
 	1    7650 4250
 	1    0    0    -1
@@
 F 2 "Resistor_SMD:R_0805_2012Metric" H 8700 4850 50  0001 C CNN
 F 3 "~" H 8700 4850 50  0001 C CNN
+F 4 "C17414" V 8700 4850 50  0001 C CNN "LCSC"
 	1    8700 4850
 	0    1    1    0
@@
 F 2 "Resistor_SMD:R_0805_2012Metric" H 6400 3750 50  0001 C CNN
 F 3 "~" H 6400 3750 50  0001 C CNN
+F 4 "C17561" V 6400 3750 50  0001 C CNN "LCSC"
 	1    6400 3750
 	0    1    1    0
@@
 F 2 "Resistor_SMD:R_0805_2012Metric" H 6150 3850 50  0001 C CNN
 F 3 "~" H 6150 3850 50  0001 C CNN
+F 4 "C17561" V 6150 3850 50  0001 C CNN "LCSC"
 	1    6150 3850
 	0    1    1    0
@@
 F 2 "Capacitor_SMD:C_0805_2012Metric" H 6400 4150 50  0001 C CNN
 F 3 "~" H 6400 4150 50  0001 C CNN
+F 4 "C28323" H 6400 4150 50  0001 C CNN "LCSC"
 	1    6400 4150
 	-1   0    0    1
@@
 	6400 4250 6400 4450
 $Comp
-L Device:C_Small C4
-U 1 1 616827A2
-P 5400 5350
-F 0 "C4" H 5492 5396 50  0000 L CNN
-F 1 "0.1uF" H 5492 5305 50  0000 L CNN
-F 2 "Capacitor_SMD:C_0805_2012Metric" H 5400 5350 50  0001 C CNN
-F 3 "~" H 5400 5350 50  0001 C CNN
-	1    5400 5350
-	1    0    0    -1
-$EndComp
-$Comp
 L Device:C_Small C5
 U 1 1 61683F91
@@
 F 2 "Capacitor_SMD:C_0805_2012Metric" H 5850 5350 50  0001 C CNN
 F 3 "~" H 5850 5350 50  0001 C CNN
+F 4 "C49678" H 5850 5350 50  0001 C CNN "LCSC"
 	1    5850 5350
 	1    0    0    -1
@@
 F 2 "Capacitor_SMD:C_0805_2012Metric" H 6300 5350 50  0001 C CNN
 F 3 "~" H 6300 5350 50  0001 C CNN
+F 4 "C49678" H 6300 5350 50  0001 C CNN "LCSC"
 	1    6300 5350
 	1    0    0    -1
@@
 F 2 "Capacitor_SMD:C_0805_2012Metric" H 6750 5350 50  0001 C CNN
 F 3 "~" H 6750 5350 50  0001 C CNN
+F 4 "C15850" H 6750 5350 50  0001 C CNN "LCSC"
 	1    6750 5350
 	1    0    0    -1
@@
 F 2 "Crystal:Crystal_SMD_3225-4Pin_3.2x2.5mm" H 6450 3050 50  0001 C CNN
 F 3 "~" H 6450 3050 50  0001 C CNN
+F 4 "C13738" H 6450 3050 50  0001 C CNN "LCSC"
 	1    6450 3050
 	0    1    1    0
@@
 F 2 "Capacitor_SMD:C_0805_2012Metric" H 6000 2850 50  0001 C CNN
 F 3 "~" H 6000 2850 50  0001 C CNN
+F 4 "C1804" V 6000 2850 50  0001 C CNN "LCSC"
 	1    6000 2850
 	0    1    1    0
@@
 F 2 "Capacitor_SMD:C_0805_2012Metric" H 6000 3250 50  0001 C CNN
 F 3 "~" H 6000 3250 50  0001 C CNN
+F 4 "C1804" V 6000 3250 50  0001 C CNN "LCSC"
 	1    6000 3250
 	0    1    1    0
@@
 F 2 "random-keyboard-parts:SKQG-1155865" H 6700 2950 50  0001 C CNN
 F 3 "~" H 6700 2950 50  0001 C CNN
+F 4 "C318884" H 6700 2750 50  0001 C CNN "LCSC"
 	1    6700 2750
 	1    0    0    -1
@@
 F 2 "Resistor_SMD:R_0805_2012Metric" H 7000 2450 50  0001 C CNN
 F 3 "~" H 7000 2450 50  0001 C CNN
+F 4 "C25804" H 7000 2450 50  0001 C CNN "LCSC"
 	1    7000 2450
 	1    0    0    -1
@@
 F 2 "random-keyboard-parts:D_SOD-123-Pretty" V 9400 4200 50  0001 C CNN
 F 3 "~" V 9400 4200 50  0001 C CNN
+F 4 "C64898" V 9400 4200 50  0001 C CNN "LCSC"
 	1    9400 4200
 	0    -1   -1   0
@@
 F 2 "random-keyboard-parts:D_SOD-123-Pretty" V 10300 3450 50  0001 C CNN
 F 3 "~" V 10300 3450 50  0001 C CNN
+F 4 "C64898" V 10300 3450 50  0001 C CNN "LCSC"
 	1    10300 3450
 	0    -1   -1   0
@@
 F 2 "random-keyboard-parts:D_SOD-123-Pretty" V 10300 4200 50  0001 C CNN
 F 3 "~" V 10300 4200 50  0001 C CNN
+F 4 "C64898" V 10300 4200 50  0001 C CNN "LCSC"
 	1    10300 4200
 	0    -1   -1   0
@@
 F 2 "random-keyboard-parts:D_SOD-123-Pretty" V 9400 3450 50  0001 C CNN
 F 3 "~" V 9400 3450 50  0001 C CNN
+F 4 "C64898" V 9400 3450 50  0001 C CNN "LCSC"
 	1    9400 3450
 	0    -1   -1   0
@@
 F 2 "Inductor_SMD:L_1206_3216Metric_Pad1.42x1.75mm_HandSolder" H 1150 2850 50  0001 C CNN
 F 3 "~" H 1150 2850 50  0001 C CNN
+F 4 "C1017" H 1150 2850 50  0001 C CNN "LCSC"
 	1    1150 2850
 	1    0    0    -1
@@
 F 2 "Package_TO_SOT_SMD:SOT-23-6" H 5100 1600 50  0001 C CNN
 F 3 "http://www.onsemi.com/pub/Collateral/SRV05-4-D.PDF" H 4400 2050 50  0001 C CNN
+F 4 "C85364" H 4400 2050 50  0001 C CNN "LCSC"
 	1    4400 2050
 	1    0    0    -1
@@
 F 2 "Fuse:Fuse_1206_3216Metric_Pad1.42x1.75mm_HandSolder" H 3950 1550 50  0001 C CNN
 F 3 "~" H 3950 1550 50  0001 C CNN
+F 4 "C70076" H 3950 1550 50  0001 C CNN "LCSC"
 	1    3950 1550
 	1    0    0    -1
@@
 F 2 "Type-C:HRO-TYPE-C-31-M-12-HandSoldering" H 1400 1650 60  0001 C CNN
 F 3 "" H 1400 1650 60  0001 C CNN
+F 4 "C165948" H 1400 1650 50  0001 C CNN "LCSC"
 	1    1400 1650
 	1    0    0    -1
@@
 F 2 "Capacitor_SMD:C_0805_2012Metric_Pad1.15x1.40mm_HandSolder" H 1800 2000 50  0001 C CNN
 F 3 "~" H 1800 2000 50  0001 C CNN
+F 4 "C23186" V 1800 2000 50  0001 C CNN "LCSC"
 	1    1800 2000
 	0    1    1    0
@@
 F 2 "Capacitor_SMD:C_0805_2012Metric_Pad1.15x1.40mm_HandSolder" H 1800 1400 50  0001 C CNN
 F 3 "~" H 1800 1400 50  0001 C CNN
+F 4 "C23186" H 1800 1400 50  0001 C CNN "LCSC"
 	1    1800 1400
 	0    1    1    0
@@
 Text Label 6900 3850 0    50   ~ 0
 DR-
+$Comp
+L Mechanical:MountingHole H1
+U 1 1 616DF6CB
+P 1250 4950
+F 0 "H1" H 1350 4996 50  0000 L CNN
+F 1 "MountingHole" H 1350 4905 50  0000 L CNN
+F 2 "MountingHole:MountingHole_2mm" H 1250 4950 50  0001 C CNN
+F 3 "~" H 1250 4950 50  0001 C CNN
+	1    1250 4950
+	1    0    0    -1
+$EndComp
+$Comp
+L Mechanical:MountingHole H4
+U 1 1 616DFE91
+P 1250 5850
+F 0 "H4" H 1350 5896 50  0000 L CNN
+F 1 "MountingHole" H 1350 5805 50  0000 L CNN
+F 2 "MountingHole:MountingHole_2mm" H 1250 5850 50  0001 C CNN
+F 3 "~" H 1250 5850 50  0001 C CNN
+	1    1250 5850
+	1    0    0    -1
+$EndComp
+$Comp
+L Mechanical:MountingHole H3
+U 1 1 616E24E7
+P 1250 5550
+F 0 "H3" H 1350 5596 50  0000 L CNN
+F 1 "MountingHole" H 1350 5505 50  0000 L CNN
+F 2 "MountingHole:MountingHole_2mm" H 1250 5550 50  0001 C CNN
+F 3 "~" H 1250 5550 50  0001 C CNN
+	1    1250 5550
+	1    0    0    -1
+$EndComp
+$Comp
+L Mechanical:MountingHole H6
+U 1 1 616E4A1C
+P 1250 6450
+F 0 "H6" H 1350 6496 50  0000 L CNN
+F 1 "MountingHole" H 1350 6405 50  0000 L CNN
+F 2 "MountingHole:MountingHole_2mm" H 1250 6450 50  0001 C CNN
+F 3 "~" H 1250 6450 50  0001 C CNN
+	1    1250 6450
+	1    0    0    -1
+$EndComp
+$Comp
+L Mechanical:MountingHole H2
+U 1 1 616F59F0
+P 1250 5250
+F 0 "H2" H 1350 5296 50  0000 L CNN
+F 1 "MountingHole" H 1350 5205 50  0000 L CNN
+F 2 "MountingHole:MountingHole_2mm" H 1250 5250 50  0001 C CNN
+F 3 "~" H 1250 5250 50  0001 C CNN
+	1    1250 5250
+	1    0    0    -1
+$EndComp
+$Comp
+L Mechanical:MountingHole H5
+U 1 1 61721932
+P 1250 6150
+F 0 "H5" H 1350 6196 50  0000 L CNN
+F 1 "MountingHole" H 1350 6105 50  0000 L CNN
+F 2 "MountingHole:MountingHole_2mm" H 1250 6150 50  0001 C CNN
+F 3 "~" H 1250 6150 50  0001 C CNN
+	1    1250 6150
+	1    0    0    -1
+$EndComp
+$Comp
+L Device:C_Small C4
+U 1 1 616827A2
+P 5400 5350
+F 0 "C4" H 5492 5396 50  0000 L CNN
+F 1 "0.1uF" H 5492 5305 50  0000 L CNN
+F 2 "Capacitor_SMD:C_0805_2012Metric" H 5400 5350 50  0001 C CNN
+F 3 "~" H 5400 5350 50  0001 C CNN
+F 4 "C49678" H 5400 5350 50  0001 C CNN "LCSC"
+	1    5400 5350
+	1    0    0    -1
+$EndComp
+NoConn ~ 4900 1950
+NoConn ~ 3900 2150
 $EndSCHEMATC

Commit message: small changes
Parts:
- F1: symbol Device:Fuse_Small -> Device:Polyfuse_Small; LCSC C70076 -> C151162
Connections:
- net +5V: now also F1.1; no longer F1.2
- net VBUS: now also F1.2; no longer F1.1

Commit message: migrate to kicad v5
Parts:
- U1: symbol MCU_Microchip_ATmega:ATmega32U4-AU -> PR-4PP-rescue:ATmega32U4-AU-MCU_Microchip_ATmega
Changed lines of the file:
@@
 EESchema Schematic File Version 4
-LIBS:PR-4PP-cache
 EELAYER 30 0
 EELAYER END
@@
 $EndDescr
 $Comp
-L MCU_Microchip_ATmega:ATmega32U4-AU U1
+L PR-4PP-rescue:ATmega32U4-AU-MCU_Microchip_ATmega U1
 U 1 1 616762F0
 P 7650 4250
